File: accelerator.kicad_pcb (KiCad board)
At the start: 2 copper layers, 466.4 x 325.6 mm, 274 parts

Commit message: impl daughterboard and plate
Parts:
- removed CL4, CR4: 4.7μF, Capacitor_SMD:C_1206_3216Metric
- removed ESDDL1, ESDDR1: ESD5Z5V0, Diode_SMD:D_SOD-523
- removed FL1, FR1: SMD0805-050-16V, Fuse:Fuse_1206_3216Metric
- removed JL1, JR1: MJ-4PP-9, MJ-4PP-9:MJ-4PP-9
- removed JL2, JR2: Conn_01x05_Pin, Connector_JST:JST_PH_S5B-PH-K_1x05_P2.00mm_Horizontal
- removed RL1, RR1: 1M, Resistor_SMD:R_1206_3216Metric
- removed RL6, RL7, RR6, RR7: 5.1k, Resistor_SMD:R_1206_3216Metric
- removed UL2, UR2: TPD4E05U06DQAR, TPD4E05U06DQAR:USON-10_L2.5-W1.0-P0.50-BL
- removed USBL1, USBR1: USB_C_Receptacle_USB2.0, Connector_USB:USB_C_Receptacle_HRO_TYPE-C-31-M-12
- added REL00_3: EncSW, Rotary_Encoder:RotaryEncoder_Alps_EC12E-Switch_Vertical_H20mm, F.Cu at (63.5, 155.2)
- added REL00_4: EncSW, Rotary_Encoder:RotaryEncoder_Alps_EC12E-Switch_Vertical_H20mm, F.Cu at (63.5, 174.3)
- moved CL1 154.7 mm to (281.1, 271.1)
- moved CL2 154.7 mm to (281.1, 274.4)
- moved CL7 154.7 mm to (286.7, 271.1)
- moved CL8 154.7 mm to (286.7, 274.4)
- moved CR2 154.7 mm to (286.7, 281.1)
- moved CR3 154.7 mm to (286.7, 284.5)
- moved CL3 154.7 mm to (281.1, 277.8)
- moved CR1 154.7 mm to (286.7, 277.8)
- moved CR5 154.7 mm to (292.4, 271.1)
- moved CR6 154.7 mm to (292.4, 274.4)
- moved CR8 154.7 mm to (292.4, 281.1)
- moved CR7 154.7 mm to (292.4, 277.8)
- moved CL5 151.7 mm to (281.1, 281.1)
- moved CL6 151.7 mm to (281.1, 284.5)
- moved LLED11 145.1 mm to (213.7, 271.9)
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Connections:
- UL1 pad 37: unconnected-(UL1-PF6-Pad37) -> RE4B
- UL1 pad 38: unconnected-(UL1-PF5-Pad38) -> RE4A
- UL1 pad 39: unconnected-(UL1-PF4-Pad39) -> RE3B
- UL1 pad 40: unconnected-(UL1-PF1-Pad40) -> RE3A
Other:
- board size 466.4 x 325.6 mm -> 3.7 x 3.3 mm
