File: accelerator.kicad_sch (KiCad schematic)
At the start: 274 parts

Commit message: impl daughterboard and plate
Parts:
- removed CL4, CR4: 4.7μF, Capacitor_SMD:C_1206_3216Metric, symbol Device:C
- removed ESDDL1, ESDDR1: ESD5Z5V0, Diode_SMD:D_SOD-523, symbol Diode:1.5KExxA
- removed FL1, FR1: SMD0805-050-16V, Fuse:Fuse_1206_3216Metric, symbol Device:Fuse
- removed JL1, JR1: MJ-4PP-9, MJ-4PP-9:MJ-4PP-9, symbol MJ-4PP-9:MJ-4PP-9
- removed JL2, JR2: Conn_01x05_Pin, Connector_JST:JST_PH_S5B-PH-K_1x05_P2.00mm_Horizontal, symbol Connector:Conn_01x05_Pin
- removed RL1, RR1: 1M, Resistor_SMD:R_1206_3216Metric, symbol Device:R
- removed RL6, RL7, RR6, RR7: 5.1k, Resistor_SMD:R_1206_3216Metric, symbol Device:R
- removed UL2, UR2: TPD4E05U06DQAR, TPD4E05U06DQAR:USON-10_L2.5-W1.0-P0.50-BL, symbol random-keyboard-parts:TPD4E05U06DQAR
- removed USBL1, USBR1: USB_C_Receptacle_USB2.0, Connector_USB:USB_C_Receptacle_HRO_TYPE-C-31-M-12, symbol Connector:USB_C_Receptacle_USB2.0_16P
- added REL00_3, REL00_4: EncSW, Rotary_Encoder:RotaryEncoder_Alps_EC12E-Switch_Vertical_H20mm, symbol Device:RotaryEncoder_Switch
Connections:
- net GNDL: now also REL00_3.C, REL00_4.C
- net lcol01: now also REL00_3.S2, REL00_4.S2
- net at DL00_18.2 (A), SWL00_25.2: now also REL00_3.S1
- net at DL00_33.2 (A), SWL00_33.2: now also REL00_4.S1
- net RE4B: now reaches UL1.37 (PF6)
- net RE4B: now also REL00_4.B
- net RE4A: now reaches UL1.38 (PF5)
- net RE4A: now also REL00_4.A
- net RE3B: now reaches UL1.39 (PF4)
- net RE3B: now also REL00_3.B
- net RE3A: now reaches UL1.40 (PF1)
- net RE3A: now also REL00_3.A
- no-connect marks 24 -> 14
Other:
- note removed: "DB L"
- note removed: "DB R"
- moved on the sheet: DL00_17, DL00_18, DL00_19, DL00_20, DL00_21, DL00_23, DL00_24, DL00_25, DL00_26, DL00_27, DL00_28, DL00_29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

Commit message: ordered
Parts:
- removed LLED16, LLED18, LLED20, LLED22, LLED24, LLED37, LLED39, RLED18, RLED20, RLED22, RLED24, RLED33, RLED35, RLED37: SK6812MINI-E, SK6812MINI-E:SK6812MINIE, symbol SK6812MINI-E:SK6812MINI-E
- added CLD1, CRD1: 4.7μF, Capacitor_SMD:C_1206_3216Metric, symbol Device:C
- added ESDDLD1, ESDDRD1: ESD5Z5V0, Diode_SMD:D_SOD-523, symbol Diode:1.5KExxA
- added FLD1, FRD1: SMD0805-050-16V, Fuse:Fuse_1206_3216Metric, symbol Device:Fuse
- added JLD1, JRD1: MJ-4PP-9, MJ-4PP-9:MJ-4PP-9, symbol MJ-4PP-9:MJ-4PP-9
- added JLD2, JRD2: Conn_01x05_Pin, Connector_JST:JST_PH_S5B-PH-K_1x05_P2.00mm_Horizontal, symbol Connector:Conn_01x05_Pin
- added LLED25, LLED26, RLED25, RLED27, RLED31: SK6812MINI-E, SK6812MINI-E:SK6812MINIE, symbol SK6812MINI-E:SK6812MINI-E
- added RLD1, RRD1: 1M, Resistor_SMD:R_1206_3216Metric, symbol Device:R
- added RLD2, RLD3, RRD2, RRD3: 5.1k, Resistor_SMD:R_1206_3216Metric, symbol Device:R
- added ULD1, URD1: TPD4E05U06DQAR, TPD4E05U06DQAR:USON-10_L2.5-W1.0-P0.50-BL, symbol random-keyboard-parts:TPD4E05U06DQAR
- added USBLD1, USBRD1: USB_C_Receptacle_USB2.0, Connector_USB:USB_C_Receptacle_HRO_TYPE-C-31-M-12, symbol Connector:USB_C_Receptacle_USB2.0_16P
- renumbered DL00_19 to DL00_18, DL00_21 to DL00_19, DL00_23 to DL00_20, DL00_25 to DL00_21, DL00_27 to DL00_22, DL00_29 to DL00_23, DL00_18 to DL00_25, DL00_20 to DL00_26, DL00_24 to DL00_28, DL00_26 to DL00_29, DL00_28 to DL00_30, DL00_30 to DL00_31, DR00_19 to DR00_18, DR00_21 to DR00_19, DR00_23 to DR00_20, DR00_25 to DR00_21, DR00_27 to DR00_22, DR00_31 to DR00_24, DR00_18 to DR00_25, DR00_20 to DR00_26, DR00_22 to DR00_27, DR00_24 to DR00_28, DR00_26 to DR00_29, DR00_28 to DR00_30, DR00_30 to DR00_31, LLED19 to LLED18, LLED21 to LLED19, LLED23 to LLED20, LLED25 to LLED21, LLED27 to LLED22, LLED29 to LLED23, LLED26 to LLED29, RLED19 to RLED18, RLED21 to RLED19, RLED23 to RLED20, RLED25 to RLED21, RLED27 to RLED22, RLED31 to RLED24
Connections:
- net +5VL: now also LLED25.1 (VDD), LLED26.1 (VDD)
- net +5VR: now also RLED25.1 (VDD), RLED27.1 (VDD), RLED31.1 (VDD)
- net GNDL: now also LLED25.3 (GND), LLED26.3 (GND)
- net GNDR: now also RLED25.3 (GND), RLED27.3 (GND), RLED31.3 (GND)
- net RE1A: now also UL1.39 (PF4); no longer UL1.25 (PD4)
- net RE1B: now also UL1.38 (PF5); no longer UL1.22 (PD5)
- net RE2A: now also UL1.37 (PF6); no longer UL1.26 (PD6)
- net RE2B: now also UL1.32 (PC7); no longer UL1.27 (PD7)
- net RE3A: now also UL1.31 (PC6); no longer UL1.40 (PF1)
- net RE3B: now also UL1.30 (PB6); no longer UL1.39 (PF4)
- net RE4A: now also UL1.29 (PB5); no longer UL1.38 (PF5)
- net RE4B: now also UL1.28 (PB4); no longer UL1.37 (PF6)
- net dataL: now also UL1.40 (PF1); no longer UL1.18 (PD0)
- net lcol01: now also UL1.25 (PD4); no longer UL1.29 (PB5)
- net lcol02: now also UL1.26 (PD6); no longer UL1.30 (PB6)
- net lcol03: now also UL1.27 (PD7); no longer UL1.12 (PB7)
- net lcol04: now also UL1.8 (PB0); no longer UL1.31 (PC6)
- net lcol05: now also UL1.9 (PB1); no longer UL1.32 (PC7)
- net lcol06: now also UL1.10 (PB2); no longer UL1.19 (PD1)
- net lcol07: now also UL1.11 (PB3); no longer UL1.20 (PD2)
- net lcol08: now also UL1.12 (PB7); no longer UL1.21 (PD3)
- net lrow01: now also UL1.22 (PD5); no longer UL1.8 (PB0)
- net lrow02: now also UL1.21 (PD3); no longer UL1.9 (PB1)
- net lrow03: now also UL1.20 (PD2); no longer UL1.10 (PB2)
- net lrow04: now also UL1.19 (PD1); no longer UL1.11 (PB3)
- net lrow05: now also UL1.18 (PD0); no longer UL1.28 (PB4)
- net rcol01: now also UR1.30 (PB6); no longer UR1.29 (PB5)
- net rcol02: now also UR1.31 (PC6); no longer UR1.30 (PB6)
- net rcol03: now also UR1.32 (PC7); no longer UR1.12 (PB7)
- net rcol04: now also UR1.36 (PF7); no longer UR1.31 (PC6)
- net rcol05: now also UR1.37 (PF6); no longer UR1.32 (PC7)
- net rcol06: now also UR1.38 (PF5); no longer UR1.19 (PD1)
- net rcol07: now also UR1.39 (PF4); no longer UR1.20 (PD2)
- net rcol08: now also UR1.40 (PF1); no longer UR1.21 (PD3)
- net rrow01: now also UR1.29 (PB5); no longer UR1.8 (PB0)
- net rrow02: now also UR1.28 (PB4); no longer UR1.9 (PB1)
- net rrow03: now also UR1.27 (PD7); no longer UR1.10 (PB2)
- net rrow04: now also UR1.26 (PD6); no longer UR1.11 (PB3)
- net rrow05: now also UR1.25 (PD4); no longer UR1.28 (PB4)
- net at LLED11.4 (DIN): now also LLED12.2 (DOUT); no longer LLED10.2 (DOUT)
- net at LLED9.2 (DOUT): now also LLED17.4 (DIN); no longer LLED10.4 (DIN)
- net at RLED16.2 (DOUT): now also RLED15.4 (DIN); no longer RLED17.4 (DIN)
- net at RLED16.4 (DIN): now also RLED8.2 (DOUT); no longer RLED15.2 (DOUT)
- net at LLED40.4 (DIN): now also LLED38.2 (DOUT)
- net at LLED15.2 (DOUT): now also LLED14.4 (DIN)
- net at LLED12.4 (DIN): now also LLED13.2 (DOUT); no longer LLED11.2 (DOUT)
- net at LLED31.2 (DOUT): now also LLED30.4 (DIN)
- net at RLED9.4 (DIN): now also RLED10.2 (DOUT); no longer RLED8.2 (DOUT)
- net at LLED13.4 (DIN): now also LLED14.2 (DOUT); no longer LLED12.2 (DOUT)
- net at LLED30.2 (DOUT): now also LLED29.4 (DIN); no longer LLED32.4 (DIN)
- net at LLED28.2 (DOUT): now also LLED26.4 (DIN); no longer LLED30.4 (DIN)
- net at LLED15.4 (DIN): now also LLED8.2 (DOUT); no longer LLED14.2 (DOUT)
- net at RLED14.2 (DOUT): now also RLED13.4 (DIN); no longer RLED15.4 (DIN)
- net at LLED36.2 (DOUT): now also LLED38.4 (DIN)
- net at RLED11.2 (DOUT): now also RLED10.4 (DIN); no longer RLED12.4 (DIN)
- net at RLED11.4 (DIN): now also RLED12.2 (DOUT); no longer RLED10.2 (DOUT)
- net at RLED29.2 (DOUT): now also RLED28.4 (DIN); no longer RLED24.4 (DIN)
- net at RLED29.4 (DIN): now also RLED30.2 (DOUT); no longer RLED22.2 (DOUT)
- net at RLED26.2 (DOUT): now also RLED25.4 (DIN); no longer RLED28.4 (DIN)
- net at RLED26.4 (DIN): now also RLED27.2 (DOUT)
- net at RLED38.4 (DIN): now also RLED36.2 (DOUT)
- net at RLED30.4 (DIN): now also RLED31.2 (DOUT); no longer RLED28.2 (DOUT)
- net at LLED31.4 (DIN): now also LLED32.2 (DOUT); no longer LLED23.2 (DOUT)
- net at RLED36.4 (DIN): now also RLED34.2 (DOUT)
- net at LLED9.4 (DIN): now also LLED10.2 (DOUT); no longer LLED8.2 (DOUT)
- net at LLED33.4 (DIN): now also LLED25.2 (DOUT); no longer LLED32.2 (DOUT)
- net at RLED34.4 (DIN): now also RLED25.2 (DOUT)
- net at RLED32.4 (DIN): now also RLED24.2 (DOUT); no longer RLED30.2 (DOUT)
- net at RLED9.2 (DOUT): now also RLED17.4 (DIN); no longer RLED10.4 (DIN)
- net at RLED14.4 (DIN): now also RLED15.2 (DOUT); no longer RLED13.2 (DOUT)
- net at RLED32.2 (DOUT): now also RLED31.4 (DIN)
- new net: LLED25.4 (DIN), LLED26.2 (DOUT)
- new net: RLED12.4 (DIN), RLED13.2 (DOUT)
- new net: RLED27.4 (DIN), RLED28.2 (DOUT)
- new net: RLED22.2 (DOUT), RLED24.4 (DIN)
- new net: LLED23.2 (DOUT), LLED32.4 (DIN)
- new net: LLED10.4 (DIN), LLED11.2 (DOUT)
- new net +5VLD: FLD1.2, JLD1.4 (D), JLD2.1 (Pin_1)
- new net +5VRD: FRD1.2, JRD1.4 (D), JRD2.1 (Pin_1)
- new net CCLD1: RLD2.2, USBLD1.A5 (CC1)
- new net CCLD2: RLD3.2, USBLD1.B5 (CC2)
- new net CCRD1: RRD2.2, USBRD1.A5 (CC1)
- new net CCRD2: RRD3.2, USBRD1.B5 (CC2)
- new net DLD+: JLD2.4 (Pin_4), ULD1.4 (D2+), ULD1.5 (D2-), ULD1.6 (NC), ULD1.7 (NC), USBLD1.A6 (D+), USBLD1.B6 (D+)
- new net DLD-: JLD2.3 (Pin_3), ULD1.1 (D1+), ULD1.10 (NC), ULD1.2 (D1-), ULD1.9 (NC), USBLD1.A7 (D-), USBLD1.B7 (D-)
- new net DRD+: JRD2.4 (Pin_4), URD1.4 (D2+), URD1.5 (D2-), URD1.6 (NC), URD1.7 (NC), USBRD1.A6 (D+), USBRD1.B6 (D+)
- new net DRD-: JRD2.3 (Pin_3), URD1.1 (D1+), URD1.10 (NC), URD1.2 (D1-), URD1.9 (NC), USBRD1.A7 (D-), USBRD1.B7 (D-)
- new net GNDLD: CLD1.1, ESDDLD1.2 (A2), JLD1.3 (C), JLD2.2 (Pin_2), RLD1.1, RLD2.1, RLD3.1, ULD1.3 (GND), ULD1.8 (GND), USBLD1.A1 (GND), USBLD1.A12 (GND), USBLD1.B1 (GND), USBLD1.B12 (GND)
- new net GNDPWRLD: CLD1.2, RLD1.2, USBLD1.S1 (SHIELD)
- new net GNDPWRRD: CRD1.2, RRD1.2, USBRD1.S1 (SHIELD)
- new net GNDRD: CRD1.1, ESDDRD1.2 (A2), JRD1.3 (C), JRD2.2 (Pin_2), RRD1.1, RRD2.1, RRD3.1, URD1.3 (GND), URD1.8 (GND), USBRD1.A1 (GND), USBRD1.A12 (GND), USBRD1.B1 (GND), USBRD1.B12 (GND)
- new net VCCLD: ESDDLD1.1 (A1), FLD1.1, USBLD1.A4 (VBUS), USBLD1.A9 (VBUS), USBLD1.B4 (VBUS), USBLD1.B9 (VBUS)
- new net VCCRD: ESDDRD1.1 (A1), FRD1.1, USBRD1.A4 (VBUS), USBRD1.A9 (VBUS), USBRD1.B4 (VBUS), USBRD1.B9 (VBUS)
- new net dataDL: JLD1.2 (B), JLD2.5 (Pin_5)
- new net dataDR: JRD1.2 (B), JRD2.5 (Pin_5)
- no-connect marks 14 -> 20
Other:
- note added: "CONNECTOR"
- note added: "ESD"
- note added: "LEFT"
- note added: "PWR"
- note added: "RIGHT"
